File: ESP32_LED.kicad_pcb (KiCad board)
At the start: 2 copper layers, 65 x 30 mm, 49 parts, among them J1 5077CR-16SMC2-BK-TR, J2 Conn_01x15, J3 Conn_01x15, J4 Servo0, J5 Servo1, J6 Servo2, J7 Servo3, J8 Iris, Q1 2SC4081, Q2 2SC4081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

Commit message: rev1.1
Parts:
- removed R15: 0, Resistor_SMD:R_0805_2012Metric
- removed R18: 300, Resistor_SMD:R_0402_1005Metric
- removed the REF** at (124.0, 74.0)
- removed the REF** at (124.0, 96.0)
- added C9: 0.1u, Capacitor_SMD:C_0402_1005Metric, F.Cu at (165.2, 95.8)
- added REF**: MountingHole_3.2mm_M3, MountingHole:MountingHole_3.2mm_M3, F.Cu at (94.0, 96.0)
- added REF**: MountingHole_3.2mm_M3, MountingHole:MountingHole_3.2mm_M3, F.Cu at (94.0, 74.0)
- C8: moved to F.Cu
- J4: value Servo0 -> Jack-DC; footprint Connector_PinHeader_2.54mm:PinHeader_1x04_P2.54mm_Vertical -> akizuki:2DC-G213-D42
- J5: value Servo1 -> JST VH; footprint Connector_PinHeader_2.54mm:PinHeader_1x04_P2.54mm_Vertical -> Connector_JST:JST_VH_B3P-VH-B_1x03_P3.96mm_Vertical
- J6: value Servo2 -> JST VH; footprint Connector_PinHeader_2.54mm:PinHeader_1x04_P2.54mm_Vertical -> Connector_JST:JST_VH_B3P-VH-B_1x03_P3.96mm_Vertical
- J7: value Servo3 -> JST VH; footprint Connector_PinHeader_2.54mm:PinHeader_1x04_P2.54mm_Vertical -> Connector_JST:JST_VH_B3P-VH-B_1x03_P3.96mm_Vertical
- J8: value Iris -> JST VH; footprint Connector_FFC-FPC:Hirose_FH12-22S-0.5SH_1x22-1MP_P0.50mm_Horizontal -> Connector_JST:JST_VH_B3P-VH-B_1x03_P3.96mm_Vertical; moved to F.Cu
- R13: value 0(NC) -> 0
- moved J8 43.0 mm to (111.2, 96.5), turned to 90 degrees
- moved J4 39.5 mm to (90.2, 85.0), turned to 90 degrees
- moved C8 23.5 mm to (105.4, 85.2), turned to 270 degrees
- moved J6 18.5 mm to (111.6, 81.6), turned to 90 degrees
- moved J5 12.0 mm to (123.2, 73.7)
- moved J7 6.36 mm to (123.2, 88.6)
- moved R13 3.81 mm to (165.0, 79.3)
- moved R8 1.04 mm to (134.1, 97.3)
- moved C3 1.02 mm to (165.2, 94.5)
- moved R1 1.02 mm to (165.2, 90.7)
- moved R3 1.02 mm to (165.2, 91.9)
- moved R4 1.02 mm to (165.2, 89.4)
- moved R10 1.02 mm to (131.6, 98.6)
- moved R11 1.02 mm to (134.1, 98.6)
- moved R2 1.02 mm to (165.2, 93.2)
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Connections:
- J1 pad A8: Net-(J1-PadA8) -> (no net)
- J1 pad B8: Net-(J1-PadB8) -> (no net)
- J2 pad 10: RST -> IO32
- J2 pad 3: D1 -> IO13
- J2 pad 4: D0 -> IO12
- J2 pad 5: D7 -> IO14
- J2 pad 6: D6 -> IO27
- J2 pad 7: D2 -> IO26
- J2 pad 8: D3 -> IO25
- J2 pad 9: CS1 -> IO33
- J3 pad 3: DC -> IO15
- J3 pad 4: WD -> IO2
- J3 pad 5: WR -> IO4
- J3 pad 6: D5 -> IO16
- J3 pad 7: D4 -> IO17
- J4 pad 1: GND -> Net-(C8-Pad1)
- J4 pad 2: Net-(J4-Pad2) -> GND
- J5 pad 1: GND -> Net-(C8-Pad1)
- J5 pad 3: Net-(C8-Pad1) -> GND
- J6 pad 1: GND -> Net-(C8-Pad1)
- J6 pad 3: Net-(C8-Pad1) -> GND
- J7 pad 1: GND -> Net-(C8-Pad1)
- J7 pad 3: Net-(C8-Pad1) -> GND
- J8 pad 1: GND -> Net-(C8-Pad1)
- J8 pad 2: RST -> Net-(J8-Pad2)
- R10 pad 1: Net-(J6-Pad2) -> Net-(J7-Pad2)
- R10 pad 2: Net-(J2-Pad12) -> IO33
- R11 pad 1: Net-(J7-Pad2) -> Net-(J8-Pad2)
- R11 pad 2: Net-(J2-Pad13) -> IO32
- R12 pad 1: D1 -> IO13
- R13 pad 2: +3V3 -> VBUS
- R8 pad 1: Net-(J4-Pad2) -> Net-(J5-Pad2)
- R8 pad 2: RST -> IO25
- R9 pad 1: Net-(J5-Pad2) -> Net-(J6-Pad2)
- R9 pad 2: Net-(J2-Pad11) -> IO26
- U1 pad 1: Net-(U1-Pad1) -> (no net)
- U1 pad 10: Net-(U1-Pad10) -> (no net)
- U1 pad 11: Net-(U1-Pad11) -> (no net)
- U1 pad 12: Net-(U1-Pad12) -> (no net)
- U1 pad 13: Net-(U1-Pad13) -> (no net)
- U1 pad 14: Net-(U1-Pad14) -> (no net)
- U1 pad 15: Net-(U1-Pad15) -> (no net)
- U1 pad 17: Net-(U1-Pad17) -> (no net)
- U1 pad 18: Net-(U1-Pad18) -> (no net)
- U1 pad 22: Net-(U1-Pad22) -> (no net)
- U1 pad 24: Net-(U1-Pad24) -> (no net)
- U1 pad 25: GND -> (no net)
- U2 pad 10: D3 -> IO25
- U2 pad 11: D2 -> IO26
- U2 pad 12: D6 -> IO27
- U2 pad 13: D7 -> IO14
- U2 pad 14: D0 -> IO12
- U2 pad 16: D1 -> IO13
- U2 pad 17: Net-(U2-Pad17) -> (no net)
- U2 pad 18: Net-(U2-Pad18) -> (no net)
- U2 pad 19: Net-(U2-Pad19) -> (no net)
- U2 pad 20: Net-(U2-Pad20) -> (no net)
- U2 pad 21: Net-(U2-Pad21) -> (no net)
- U2 pad 22: Net-(U2-Pad22) -> (no net)
- U2 pad 23: DC -> IO15
- U2 pad 24: WD -> IO2
- U2 pad 26: WR -> IO4
- U2 pad 27: D5 -> IO16
- U2 pad 28: D4 -> IO17
- U2 pad 32: Net-(U2-Pad32) -> (no net)
- U2 pad 8: RST -> IO32
- U2 pad 9: CS1 -> IO33
Routing:
- net Net-(C8-Pad1): track 62.2 -> 214.4 mm, vias 5 -> 6
- net D1: track 48.2 -> 0.00 mm, vias 1 -> 0
- net RST: track 40.9 -> 0.00 mm, vias 2 -> 0
- net IO26: track 0.00 -> 33.6 mm, vias 0 -> 1
- net D0: track 31.7 -> 0.00 mm, vias 1 -> 0
- net IO13: track 0.00 -> 29.3 mm
- net IO25: track 0.00 -> 27.8 mm, vias 0 -> 1
- net IO33: track 0.00 -> 27.3 mm, vias 0 -> 1
- net Net-(J8-Pad2): track 0.00 -> 27.0 mm
- net D7: track 25.7 -> 0.00 mm, vias 1 -> 0
- net GND: track 136.6 -> 111.5 mm
- net WD: track 24.6 -> 0.00 mm, vias 1 -> 0
- net DC: track 24.6 -> 0.00 mm, vias 1 -> 0
- net Net-(J6-Pad2): track 13.9 -> 37.4 mm
- net D6: track 23.4 -> 0.00 mm, vias 1 -> 0
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Other:
- board size 65 x 30 mm -> 95 x 30 mm
- net class Default: clearance 0.2 -> 0.16; trace_width 0.25 -> 0.16
- rule trace_clearance: 0.2 -> 0.16
- rule via_min_drill: 0.4 -> 0.3
- rule via_min_size: 0.5 -> 0.4
- board text added: "2021.04.18"
- board text removed: "2021.02.22"
- board text removed: "5V"
- board text removed: "Majoka LCD"
- board text removed: "Sig"
