File: ESP32_LED.kicad_pcb (KiCad board)
At the start: 2 copper layers, 65 x 30 mm, 49 parts, among them J1 5077CR-16SMC2-BK-TR, J2 Conn_01x15, J3 Conn_01x15, J4 Servo0, J5 Servo1, J6 Servo2, J7 Servo3, J8 Iris, Q1 2SC4081, Q2 2SC4081, SW1 MODE, SW2 RESET, U1 CP2104-F03-GM, U2 ESP-WROOM-32, U3 TC2117

Commit message: rev1.2
Parts:
- removed J7: Servo3, Connector_PinHeader_2.54mm:PinHeader_1x04_P2.54mm_Vertical
- removed J8: Iris, Connector_FFC-FPC:Hirose_FH12-22S-0.5SH_1x22-1MP_P0.50mm_Horizontal
- removed R10, R11, R18: 300, Resistor_SMD:R_0402_1005Metric
- removed R13: 0(NC), Resistor_SMD:R_0805_2012Metric
- removed R14, R15: 0, Resistor_SMD:R_0805_2012Metric
- removed the REF** at (124.0, 74.0)
- removed the REF** at (124.0, 96.0)
- added ?: , universal:universal-1pin, F.Cu at (119.4, 73.7)
- added ?: , universal:universal-1pin, F.Cu at (129.5, 96.5)
- added ?: , universal:universal-1pin, F.Cu at (119.4, 96.5)
- added ?: , universal:universal-1pin, F.Cu at (121.9, 96.5)
- added ?: , universal:universal-1pin, F.Cu at (127.0, 96.5)
- added ?: , universal:universal-1pin, F.Cu at (114.3, 96.5)
- added ?: , universal:universal-1pin, F.Cu at (116.8, 96.5)
- added ?: , universal:universal-1pin, F.Cu at (124.5, 96.5)
- added ?: , universal:universal-1pin, F.Cu at (129.5, 94.0)
- added ?: , universal:universal-1pin, F.Cu at (127.0, 94.0)
- added ?: , universal:universal-1pin, F.Cu at (116.8, 94.0)
- added ?: , universal:universal-1pin, F.Cu at (124.5, 73.7)
- added ?: , universal:universal-1pin, F.Cu at (132.1, 94.0)
- added ?: , universal:universal-1pin, F.Cu at (121.9, 94.0)
- added ?: , universal:universal-1pin, F.Cu at (119.4, 94.0)
- added ?: , universal:universal-1pin, F.Cu at (114.3, 94.0)
- added ?: , universal:universal-1pin, F.Cu at (116.8, 91.4)
- added ?: , universal:universal-1pin, F.Cu at (124.5, 88.9)
- added ?: , universal:universal-1pin, F.Cu at (114.3, 88.9)
- added ?: , universal:universal-1pin, F.Cu at (116.8, 88.9)
- added ?: , universal:universal-1pin, F.Cu at (114.3, 86.4)
- added ?: , universal:universal-1pin, F.Cu at (127.0, 88.9)
- added ?: , universal:universal-1pin, F.Cu at (114.3, 73.7)
- added ?: , universal:universal-1pin, F.Cu at (129.5, 86.4)
- added ?: , universal:universal-1pin, F.Cu at (127.0, 91.4)
- added ?: , universal:universal-1pin, F.Cu at (129.5, 91.4)
- added ?: , universal:universal-1pin, F.Cu at (132.1, 88.9)
- added ?: , universal:universal-1pin, F.Cu at (121.9, 88.9)
- added ?: , universal:universal-1pin, F.Cu at (119.4, 88.9)
- added ?: , universal:universal-1pin, F.Cu at (132.1, 91.4)
- added ?: , universal:universal-1pin, F.Cu at (121.9, 91.4)
- added ?: , universal:universal-1pin, F.Cu at (119.4, 91.4)
- added ?: , universal:universal-1pin, F.Cu at (132.1, 86.4)
- added ?: , universal:universal-1pin, F.Cu at (129.5, 73.7)
- added ?: , universal:universal-1pin, F.Cu at (119.4, 86.4)
- added ?: , universal:universal-1pin, F.Cu at (127.0, 86.4)
- added ?: , universal:universal-1pin, F.Cu at (116.8, 86.4)
- added ?: , universal:universal-1pin, F.Cu at (124.5, 86.4)
- added ?: , universal:universal-1pin, F.Cu at (124.5, 94.0)
- added ?: , universal:universal-1pin, F.Cu at (129.5, 88.9)
- added ?: , universal:universal-1pin, F.Cu at (124.5, 91.4)
- added ?: , universal:universal-1pin, F.Cu at (114.3, 91.4)
- added ?: , universal:universal-1pin, F.Cu at (121.9, 86.4)
- added ?: , universal:universal-1pin, F.Cu at (116.8, 83.8)
- added ?: , universal:universal-1pin, F.Cu at (132.1, 73.7)
- added ?: , universal:universal-1pin, F.Cu at (127.0, 83.8)
- added ?: , universal:universal-1pin, F.Cu at (129.5, 83.8)
- added ?: , universal:universal-1pin, F.Cu at (132.1, 83.8)
- added ?: , universal:universal-1pin, F.Cu at (121.9, 83.8)
- added ?: , universal:universal-1pin, F.Cu at (119.4, 83.8)
- added ?: , universal:universal-1pin, F.Cu at (124.5, 83.8)
- added ?: , universal:universal-1pin, F.Cu at (114.3, 83.8)
- added ?: , universal:universal-1pin, F.Cu at (124.5, 81.3)
- added ?: , universal:universal-1pin, F.Cu at (114.3, 81.3)
- added ?: , universal:universal-1pin, F.Cu at (116.8, 81.3)
- added ?: , universal:universal-1pin, F.Cu at (127.0, 73.7)
- added ?: , universal:universal-1pin, F.Cu at (127.0, 81.3)
- added ?: , universal:universal-1pin, F.Cu at (132.1, 81.3)
- added ?: , universal:universal-1pin, F.Cu at (121.9, 81.3)
- added ?: , universal:universal-1pin, F.Cu at (119.4, 81.3)
- added ?: , universal:universal-1pin, F.Cu at (129.5, 81.3)
- added ?: , universal:universal-1pin, F.Cu at (114.3, 78.7)
- added ?: , universal:universal-1pin, F.Cu at (129.5, 78.7)
- added ?: , universal:universal-1pin, F.Cu at (132.1, 78.7)
- added ?: , universal:universal-1pin, F.Cu at (119.4, 78.7)
- added ?: , universal:universal-1pin, F.Cu at (127.0, 78.7)
- added ?: , universal:universal-1pin, F.Cu at (121.9, 73.7)
- added ?: , universal:universal-1pin, F.Cu at (116.8, 78.7)
- added ?: , universal:universal-1pin, F.Cu at (124.5, 78.7)
- added ?: , universal:universal-1pin, F.Cu at (121.9, 78.7)
- added ?: , universal:universal-1pin, F.Cu at (132.1, 76.2)
- added ?: , universal:universal-1pin, F.Cu at (129.5, 76.2)
- added ?: , universal:universal-1pin, F.Cu at (127.0, 76.2)
- added ?: , universal:universal-1pin, F.Cu at (124.5, 76.2)
- added ?: , universal:universal-1pin, F.Cu at (121.9, 76.2)
- added ?: , universal:universal-1pin, F.Cu at (119.4, 76.2)
- added ?: , universal:universal-1pin, F.Cu at (116.8, 76.2)
- added ?: , universal:universal-1pin, F.Cu at (116.8, 73.7)
- added ?: , universal:universal-1pin, F.Cu at (114.3, 76.2)
- added ?: , universal:universal-1pin, F.Cu at (132.1, 96.5)
- added C9: 0.1u, Capacitor_SMD:C_0402_1005Metric, F.Cu at (165.2, 95.8)
- added D4: RBS5LAM40ATR, RS:SOD-128, F.Cu at (165.1, 77.9)
- added REF**: MountingHole_3.2mm_M3, MountingHole:MountingHole_3.2mm_M3, F.Cu at (94.0, 96.0)
- added REF**: MountingHole_3.2mm_M3, MountingHole:MountingHole_3.2mm_M3, F.Cu at (94.0, 74.0)
- J4: value Servo0 -> Jack-DC; footprint Connector_PinHeader_2.54mm:PinHeader_1x04_P2.54mm_Vertical -> akizuki:2DC-G213-D42
- J5: value Servo1 -> JST VH; footprint Connector_PinHeader_2.54mm:PinHeader_1x04_P2.54mm_Vertical -> Connector_JST:JST_VH_B3P-VH-B_1x03_P3.96mm_Vertical
- J6: value Servo2 -> JST VH; footprint Connector_PinHeader_2.54mm:PinHeader_1x04_P2.54mm_Vertical -> Connector_JST:JST_VH_B3P-VH-B_1x03_P3.96mm_Vertical
- moved J4 42.5 mm to (87.2, 85.0), turned to 90 degrees
- moved C8 32.1 mm to (96.5, 85.1), turned to 180 degrees
- moved J5 23.6 mm to (108.0, 74.1)
- moved J6 21.6 mm to (108.0, 88.0)
- moved R8 2.17 mm to (134.1, 99.2)
- moved R9 2.16 mm to (131.6, 99.2)
- moved C7 1.32 mm to (167.6, 76.7)
- moved C3 1.02 mm to (165.2, 94.5)
- moved R1 1.02 mm to (165.2, 90.7)
- moved R3 1.02 mm to (165.2, 91.9)
- moved R4 1.02 mm to (165.2, 89.4)
- moved R2 1.02 mm to (165.2, 93.2)
- moved R7 0.91 mm to (164.9, 84.5)
- moved C4 0.91 mm to (164.9, 85.7)
- moved C5 0.76 mm to (165.2, 87.4)
Connections:
- net CS1 renamed IO33
- net D0 renamed IO12
- net D1 renamed IO13
- net D4 renamed IO17
- net D5 renamed IO16
- net D6 renamed IO27
- net D7 renamed IO14
- net DC renamed IO15
- net WD renamed IO2
- net WR renamed IO4
- J2 pad 10: RST -> IO32
- J2 pad 7: D2 -> IO26
- J2 pad 8: D3 -> IO25
- J4 pad 1: GND -> Net-(C8-Pad1)
- J4 pad 2: Net-(J4-Pad2) -> GND
- J5 pad 1: GND -> Net-(C8-Pad1)
- J5 pad 3: Net-(C8-Pad1) -> GND
- J6 pad 1: GND -> Net-(C8-Pad1)
- J6 pad 3: Net-(C8-Pad1) -> GND
- R8 pad 1: Net-(J4-Pad2) -> Net-(J5-Pad2)
- R8 pad 2: RST -> IO25
- R9 pad 1: Net-(J5-Pad2) -> Net-(J6-Pad2)
- R9 pad 2: Net-(J2-Pad11) -> IO26
- U1 pad 25: GND -> (no net)
- U2 pad 10: D3 -> IO25
- U2 pad 11: D2 -> IO26
- U2 pad 8: RST -> IO32
Routing:
- net Net-(C8-Pad1): track 62.2 -> 103.4 mm, vias 5 -> 6
- net RST: track 40.9 -> 0.00 mm, vias 2 -> 0
- net IO26: track 0.00 -> 35.3 mm, vias 0 -> 1
- net IO25: track 0.00 -> 29.7 mm, vias 0 -> 1
- net Net-(J5-Pad2): track 18.0 -> 45.2 mm
- net D2: track 22.8 -> 0.00 mm, vias 1 -> 0
- net IO12: track 31.7 -> 9.02 mm, vias 1 -> 0
- net Net-(J4-Pad2): track 22.4 -> 0.00 mm
- net D3: track 21.3 -> 0.00 mm, vias 1 -> 0
- net Net-(J2-Pad11): track 24.3 -> 5.32 mm, vias 1 -> 0
- net IO13: track 48.2 -> 29.3 mm, vias 1 -> 0
- net IO14: track 25.7 -> 7.65 mm, vias 1 -> 0
- net IO27: track 23.4 -> 6.38 mm, vias 1 -> 0
- net VBUS: track 75.2 -> 58.3 mm, vias 5 -> 4
- net Net-(J2-Pad12): track 22.4 -> 6.01 mm, vias 1 -> 0
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Other:
- board size 65 x 30 mm -> 95 x 30 mm
- net class Default: clearance 0.2 -> 0.16; trace_width 0.25 -> 0.16
- rule trace_clearance: 0.2 -> 0.16
- rule via_min_drill: 0.4 -> 0.3
- rule via_min_size: 0.5 -> 0.4
- board text added: "2021.08.11 ver 1.2"
- board text removed: "2021.02.22"
- board text removed: "5V"
- board text removed: "Majoka LCD"
- board text removed: "Sig"
